File: teensy.sch (KiCad schematic (older format))
At the start: 2 parts, among them J1 Conn_01x10, U1 Teensy++

Commit message: Add holes for Teensy
Parts:
- U1: footprint teensy:Teensy2.0++Pads -> teensy:Teensy2.0++
Changed lines of the file:
@@
 EESchema Schematic File Version 4
-LIBS:t430-teensypp-cache
 EELAYER 30 0
 EELAYER END
@@
 F 0 "U1" H 5950 2315 50  0000 C CNN
 F 1 "Teensy++" H 5950 2224 50  0000 C CNN
-F 2 "teensy:Teensy2.0++Pads" H 6250 2150 50  0001 C CNN
+F 2 "teensy:Teensy2.0++" H 6250 2150 50  0001 C CNN
 F 3 "" H 6250 2150 50  0001 C CNN
 	1    5750 2150
@@
 	8750 3850 8950 3850
 $Comp
-L power:GND #PWR?
+L power:GND #PWR0131
 U 1 1 5D524C67
 P 8550 3950
-F 0 "#PWR?" H 8550 3700 50  0001 C CNN
+F 0 "#PWR0131" H 8550 3700 50  0001 C CNN
 F 1 "GND" H 8555 3777 50  0000 C CNN
 F 2 "" H 8550 3950 50  0001 C CNN
